Commit message: Write joint angle reading and simulation.

File: ctm_mpt_image/urdf/ctm_mpt.xacro (robot description, xacro)
@@ -4,6 +4,6 @@
   <!-- Constants. -->
   <xacro:property name="PI" value="3.1415926535897931"/>
-  <xacro:property name="LOWER" value="${-PI/9}"/>
-  <xacro:property name="UPPER" value="${PI/9}"/>
+  <xacro:property name="LOWER" value="${-PI/2}"/>
+  <xacro:property name="UPPER" value="${PI/2}"/>
   <xacro:property name="EFFORT" value="100"/>
   <xacro:property name="VELOCITY" value="1.0"/>
@@ -189,5 +189,5 @@
     <parent link="Seg1"/>
     <child link="UnvJnt2"/>
-    <axis xyz="0 1 0"/>
+    <axis xyz="1 0 0"/>
     <limit
       lower="${LOWER}"
@@ -201,5 +201,5 @@
       <origin
         xyz="1.86533836377123E-07 -1.0468209887815E-06 0.0639997244435651"
-        rpy="0 0 0"/>
+        rpy="0 0 ${PI/2}"/>
       <mass value="0.525659230606409"/>
       <inertia
@@ -214,5 +214,5 @@
       <origin
         xyz="0 0 0"
-        rpy="0 0 0"/>
+        rpy="0 0 ${PI/2}"/>
       <geometry>
         <mesh filename="package://ctm_mpt_image/meshes/Seg.stl"/>
@@ -225,5 +225,5 @@
       <origin
         xyz="0 0 0"
-        rpy="0 0 0"/>
+        rpy="0 0 ${PI/2}"/>
       <geometry>
         <mesh filename="package://ctm_mpt_image/meshes/Seg.stl"/>
@@ -238,5 +238,5 @@
     <parent link="UnvJnt2"/>
     <child link="Seg2"/>
-    <axis xyz="1 0 0"/>
+    <axis xyz="0 1 0"/>
     <limit
       lower="${LOWER}"
@@ -385,5 +385,5 @@
     <parent link="Seg3"/>
     <child link="UnvJnt4"/>
-    <axis xyz="0 1 0"/>
+    <axis xyz="1 0 0"/>
     <limit
       lower="${LOWER}"
@@ -397,5 +397,5 @@
       <origin
         xyz="1.86533835044855E-07 -1.04682098811537E-06 0.0639997244435642"
-        rpy="0 0 0"/>
+        rpy="0 0 ${PI/2}"/>
       <mass value="0.525659230606464"/>
       <inertia
@@ -410,5 +410,5 @@
       <origin
         xyz="0 0 0"
-        rpy="0 0 0"/>
+        rpy="0 0 ${PI/2}"/>
       <geometry>
         <mesh filename="package://ctm_mpt_image/meshes/Seg.stl"/>
@@ -421,5 +421,5 @@
       <origin
         xyz="0 0 0"
-        rpy="0 0 0"/>
+        rpy="0 0 ${PI/2}"/>
       <geometry>
         <mesh filename="package://ctm_mpt_image/meshes/Seg.stl"/>
@@ -434,5 +434,5 @@
     <parent link="UnvJnt4"/>
     <child link="Seg4"/>
-    <axis xyz="1 0 0"/>
+    <axis xyz="0 1 0"/>
     <limit
       lower="${LOWER}"
@@ -581,5 +581,5 @@
     <parent link="Seg5"/>
     <child link="UnvJnt6"/>
-    <axis xyz="0 1 0"/>
+    <axis xyz="1 0 0"/>
     <limit
       lower="${LOWER}"
@@ -593,5 +593,5 @@
       <origin
         xyz="1.86533836377123E-07 -1.04682098855946E-06 0.0639997244435645"
-        rpy="0 0 0"/>
+        rpy="0 0 ${PI/2}"/>
       <mass value="0.525659230606459"/>
       <inertia
@@ -606,5 +606,5 @@
       <origin
         xyz="0 0 0"
-        rpy="0 0 0"/>
+        rpy="0 0 ${PI/2}"/>
       <geometry>
         <mesh filename="package://ctm_mpt_image/meshes/Seg.stl"/>
@@ -617,5 +617,5 @@
       <origin
         xyz="0 0 0"
-        rpy="0 0 0"/>
+        rpy="0 0 ${PI/2}"/>
       <geometry>
         <mesh filename="package://ctm_mpt_image/meshes/Seg.stl"/>
@@ -630,5 +630,5 @@
     <parent link="UnvJnt6"/>
     <child link="Seg6"/>
-    <axis xyz="1 0 0"/>
+    <axis xyz="0 1 0"/>
     <limit
       lower="${LOWER}"
@@ -777,5 +777,5 @@
     <parent link="Seg7"/>
     <child link="UnvJnt8"/>
-    <axis xyz="0 1 0"/>
+    <axis xyz="1 0 0"/>
     <limit
       lower="${LOWER}"
@@ -789,5 +789,5 @@
       <origin
         xyz="1.86533834600766E-07 -1.04682098811537E-06 0.0639997244435644"
-        rpy="0 0 0"/>
+        rpy="0 0 ${PI/2}"/>
       <mass value="0.525659230606457"/>
       <inertia
@@ -802,5 +802,5 @@
       <origin
         xyz="0 0 0"
-        rpy="0 0 0"/>
+        rpy="0 0 ${PI/2}"/>
       <geometry>
         <mesh filename="package://ctm_mpt_image/meshes/Seg.stl"/>
@@ -813,5 +813,5 @@
       <origin
         xyz="0 0 0"
-        rpy="0 0 0"/>
+        rpy="0 0 ${PI/2}"/>
       <geometry>
         <mesh filename="package://ctm_mpt_image/meshes/Seg.stl"/>
@@ -826,5 +826,5 @@
     <parent link="UnvJnt8"/>
     <child link="Seg8"/>
-    <axis xyz="1 0 0"/>
+    <axis xyz="0 1 0"/>
     <limit
       lower="${LOWER}"

Commit message: Qiu Ke urdf motion

File: ctm_mpt_image/urdf/ctm_mpt.xacro (robot description, xacro)
@@ -931,3 +931,26 @@
       velocity="${VELOCITY}"/>
   </joint>
+  <link name="Tip">
+    <inertial>
+      <origin
+        xyz="5.78568388753808E-07 5.03623603487213E-07 0.0608602283267965"
+        rpy="0 0 0"/>
+      <mass value="0.497271341157921"/>
+      <inertia
+        ixx="0.00089124527277552"
+        ixy="-1.54419534730238E-09"
+        ixz="-1.30176586244889E-08"
+        iyy="0.000934969477700439"
+        iyz="1.62415264433302E-09"
+        izz="0.000719370850011746"/>
+    </inertial>
+  </link>
+  <joint name="S9T" type="fixed">
+    <origin
+      xyz="0 0 0.128"
+      rpy="0 0 0"/>
+    <parent link="Seg9_Head"/>
+    <child link="Tip"/>
+    <axis xyz="1 0 0"/>
+  </joint>
 </robot>
